File: pwr-level.sch (KiCad schematic (older format))
At the start: 15 parts, among them J1 Conn_01x02, J2 Conn_01x01, J3 Conn_01x01, U1 L78L05_SOT89, U2 ATtiny13-20SU, U3 MAX7219, U4 KCSA02-106, U5 KCSA02-106, U6 KCSA02-106

Commit message: Schematics/PCB update
- Added current limit resistor for LED display
- Updated PCB layout
Parts:
- added R5: 1kOm, Resistor_SMD:R_1206_3216Metric, symbol Device:R_Small
Connections:
- net +5V: now also R5.2; no longer U3.18 (ISET)
- new net: R5.1, U3.18 (ISET)
Changed lines of the file:
@@
 Wire Wire Line
 	4550 1900 4550 2050
-$Comp
-L power:+5V #PWR0108
-U 1 1 5FD8916D
-P 6400 2600
-F 0 "#PWR0108" H 6400 2450 50  0001 C CNN
-F 1 "+5V" V 6415 2728 50  0000 L CNN
-F 2 "" H 6400 2600 50  0001 C CNN
-F 3 "" H 6400 2600 50  0001 C CNN
-	1    6400 2600
-	0    -1   -1   0
-$EndComp
 Wire Wire Line
 	7000 2400 7000 2250
 Wire Wire Line
-	7000 2250 6500 2250
-Wire Wire Line
-	6500 2250 6500 2600
-Wire Wire Line
-	6500 2600 6400 2600
-Wire Wire Line
-	6600 2600 6500 2600
-Connection ~ 6500 2600
+	7000 2250 6750 2250
 $Comp
 L Device:R_Small R4
@@
 NoConn ~ 650  1750
 NoConn ~ 7400 4100
+$Comp
+L Device:R_Small R5
+U 1 1 60246818
+P 6500 2400
+F 0 "R5" V 6304 2400 50  0000 C CNN
+F 1 "1kOm" V 6395 2400 50  0000 C CNN
+F 2 "Resistor_SMD:R_1206_3216Metric" H 6500 2400 50  0001 C CNN
+F 3 "~" H 6500 2400 50  0001 C CNN
+	1    6500 2400
+	-1   0    0    1
+$EndComp
+Wire Wire Line
+	6500 2250 6500 2300
+Wire Wire Line
+	6500 2500 6500 2600
+Wire Wire Line
+	6500 2600 6600 2600
+$Comp
+L power:+5V #PWR0103
+U 1 1 6024DD6E
+P 6750 2150
+F 0 "#PWR0103" H 6750 2000 50  0001 C CNN
+F 1 "+5V" V 6765 2278 50  0000 L CNN
+F 2 "" H 6750 2150 50  0001 C CNN
+F 3 "" H 6750 2150 50  0001 C CNN
+	1    6750 2150
+	1    0    0    -1
+$EndComp
+Wire Wire Line
+	6750 2150 6750 2250
+Connection ~ 6750 2250
+Wire Wire Line
+	6750 2250 6500 2250
 Wire Bus Line
 	7750 3500 7750 6100

Commit message: Schematics update
- Added 1pin markers for CPU/LED driver
- Updated b.Cu/f.Cu GND fill
Parts:
- R5: value 1kOm -> 10kOm
Changed lines of the file:
@@
 P 6500 2400
 F 0 "R5" V 6304 2400 50  0000 C CNN
-F 1 "1kOm" V 6395 2400 50  0000 C CNN
+F 1 "10kOm" V 6395 2400 50  0000 C CNN
 F 2 "Resistor_SMD:R_1206_3216Metric" H 6500 2400 50  0001 C CNN
 F 3 "~" H 6500 2400 50  0001 C CNN

Commit message: Resistor devider values update for ADC
Parts:
- R1: value 33 -> 30kOm
- R2: value 30 -> 20kOm
- R4: value 33k -> 4.7kOm
Changed lines of the file:
@@
 P 5600 3450
 F 0 "R1" V 5404 3450 50  0000 C CNN
-F 1 "33" V 5495 3450 50  0000 C CNN
+F 1 "30kOm" V 5495 3450 50  0000 C CNN
 F 2 "Resistor_SMD:R_1206_3216Metric" H 5600 3450 50  0001 C CNN
 F 3 "~" H 5600 3450 50  0001 C CNN
@@
 P 5200 3450
 F 0 "R2" V 5004 3450 50  0000 C CNN
-F 1 "30" V 5095 3450 50  0000 C CNN
+F 1 "20kOm" V 5095 3450 50  0000 C CNN
 F 2 "Resistor_SMD:R_1206_3216Metric" H 5200 3450 50  0001 C CNN
 F 3 "~" H 5200 3450 50  0001 C CNN
@@
 P 5450 2950
 F 0 "R4" V 5254 2950 50  0000 C CNN
-F 1 "33k" V 5345 2950 50  0000 C CNN
+F 1 "4.7kOm" V 5345 2950 50  0000 C CNN
 F 2 "Resistor_SMD:R_1206_3216Metric" H 5450 2950 50  0001 C CNN
 F 3 "~" H 5450 2950 50  0001 C CNN
